Commit message: Ongoing : lecture content

File: test_description/urdf/fusionbot.urdf (robot description, URDF)
Before this commit: robot fusionbot, 5 links, 4 joints
Links:
- link base_link: geometry collision mesh filename=/home/kimsooyoung/ros2_ws/install/test_description/share/te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 scale=0.001 0.001 0.001; visual mesh filename=/home/kimsooyoung/ros2_ws/install/test_description/share/te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 scale=0.001 0.001 0.001
- link left_wheel_1: geometry collision mesh filename=/home/kimsooyoung/ros2_ws/install/test_description/share/te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 scale=0.001 0.001 0.001; visual mesh filename=/home/kimsooyoung/ros2_ws/install/test_description/share/te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 scale=0.001 0.001 0.001
- link lidar_1: geometry collision mesh filename=/home/kimsooyoung/ros2_ws/install/test_description/share/te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 scale=0.001 0.001 0.001; visual mesh filename=/home/kimsooyoung/ros2_ws/install/test_description/share/te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 scale=0.001 0.001 0.001
- link right_wheel_1: geometry collision mesh filename=/home/kimsooyoung/ros2_ws/install/test_description/share/te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 scale=0.001 0.001 0.001; visual mesh filename=/home/kimsooyoung/ros2_ws/install/test_description/share/te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 scale=0.001 0.001 0.001
