Commit message: model uri => pkg uri

File: test_description/urdf/fusionbot.urdf.xacro (robot description, xacro)
@@ -14,5 +14,5 @@
     <origin rpy="0 0 0" xyz="0 0 0"/>
     <geometry>
-      <mesh filename="model://test_description/meshes/base_link.stl" scale="0.001 0.001 0.001"/>
+      <mesh filename="package://test_description/meshes/base_link.stl" scale="0.001 0.001 0.001"/>
     </geometry>
     <material name="silver"/>
@@ -21,5 +21,5 @@
     <origin rpy="0 0 0" xyz="0 0 0"/>
     <geometry>
-      <mesh filename="model://test_description/meshes/base_link.stl" scale="0.001 0.001 0.001"/>
+      <mesh filename="package://test_description/meshes/base_link.stl" scale="0.001 0.001 0.001"/>
     </geometry>
   </collision>
@@ -34,5 +34,5 @@
     <origin rpy="0 0 0" xyz="-0.05 -0.0 -0.11"/>
     <geometry>
-      <mesh filename="model://test_description/meshes/lidar_1.stl" scale="0.001 0.001 0.001"/>
+      <mesh filename="package://test_description/meshes/lidar_1.stl" scale="0.001 0.001 0.001"/>
     </geometry>
     <material name="silver"/>
@@ -41,5 +41,5 @@
     <origin rpy="0 0 0" xyz="-0.05 -0.0 -0.11"/>
     <geometry>
-      <mesh filename="model://test_description/meshes/lidar_1.stl" scale="0.001 0.001 0.001"/>
+      <mesh filename="package://test_description/meshes/lidar_1.stl" scale="0.001 0.001 0.001"/>
     </geometry>
   </collision>
@@ -54,5 +54,5 @@
     <origin rpy="0 0 0" xyz="-0.0 0.1 -0.05"/>
     <geometry>
-      <mesh filename="model://test_description/meshes/right_wheel_1.stl" scale="0.001 0.001 0.001"/>
+      <mesh filename="package://test_description/meshes/right_wheel_1.stl" scale="0.001 0.001 0.001"/>
     </geometry>
     <material name="silver"/>
@@ -61,5 +61,5 @@
     <origin rpy="0 0 0" xyz="-0.0 0.1 -0.05"/>
     <geometry>
-      <mesh filename="model://test_description/meshes/right_wheel_1.stl" scale="0.001 0.001 0.001"/>
+      <mesh filename="package://test_description/meshes/right_wheel_1.stl" scale="0.001 0.001 0.001"/>
     </geometry>
   </collision>
@@ -74,5 +74,5 @@
     <origin rpy="0 0 0" xyz="-0.0 -0.1 -0.05"/>
     <geometry>
-      <mesh filename="model://test_description/meshes/left_wheel_1.stl" scale="0.001 0.001 0.001"/>
+      <mesh filename="package://test_description/meshes/left_wheel_1.stl" scale="0.001 0.001 0.001"/>
     </geometry>
     <material name="silver"/>
@@ -81,5 +81,5 @@
     <origin rpy="0 0 0" xyz="-0.0 -0.1 -0.05"/>
     <geometry>
-      <mesh filename="model://test_description/meshes/left_wheel_1.stl" scale="0.001 0.001 0.001"/>
+      <mesh filename="package://test_description/meshes/left_wheel_1.stl" scale="0.001 0.001 0.001"/>
     </geometry>
   </collision>

Commit message: ongoing : gazebo spawn

File: test_description/urdf/fusionbot.urdf.xacro (robot description, xacro)
@@ -14,5 +14,5 @@
     <origin rpy="0 0 0" xyz="0 0 0"/>
     <geometry>
-      <mesh filename="package://test_description/meshes/base_link.stl" scale="0.001 0.001 0.001"/>
+      <mesh filename="$(find test_description)/meshes/base_link.stl" scale="0.001 0.001 0.001"/>
     </geometry>
     <material name="silver"/>
@@ -21,5 +21,5 @@
     <origin rpy="0 0 0" xyz="0 0 0"/>
     <geometry>
-      <mesh filename="package://test_description/meshes/base_link.stl" scale="0.001 0.001 0.001"/>
+      <mesh filename="$(find test_description)/meshes/base_link.stl" scale="0.001 0.001 0.001"/>
     </geometry>
   </collision>
@@ -34,5 +34,5 @@
     <origin rpy="0 0 0" xyz="-0.05 -0.0 -0.11"/>
     <geometry>
-      <mesh filename="package://test_description/meshes/lidar_1.stl" scale="0.001 0.001 0.001"/>
+      <mesh filename="$(find test_description)/meshes/lidar_1.stl" scale="0.001 0.001 0.001"/>
     </geometry>
     <material name="silver"/>
@@ -41,5 +41,5 @@
     <origin rpy="0 0 0" xyz="-0.05 -0.0 -0.11"/>
     <geometry>
-      <mesh filename="package://test_description/meshes/lidar_1.stl" scale="0.001 0.001 0.001"/>
+      <mesh filename="$(find test_description)/meshes/lidar_1.stl" scale="0.001 0.001 0.001"/>
     </geometry>
   </collision>
@@ -54,5 +54,5 @@
     <origin rpy="0 0 0" xyz="-0.0 0.1 -0.05"/>
     <geometry>
-      <mesh filename="package://test_description/meshes/right_wheel_1.stl" scale="0.001 0.001 0.001"/>
+      <mesh filename="$(find test_description)/meshes/right_wheel_1.stl" scale="0.001 0.001 0.001"/>
     </geometry>
     <material name="silver"/>
@@ -61,5 +61,5 @@
     <origin rpy="0 0 0" xyz="-0.0 0.1 -0.05"/>
     <geometry>
-      <mesh filename="package://test_description/meshes/right_wheel_1.stl" scale="0.001 0.001 0.001"/>
+      <mesh filename="$(find test_description)/meshes/right_wheel_1.stl" scale="0.001 0.001 0.001"/>
     </geometry>
   </collision>
@@ -74,5 +74,5 @@
     <origin rpy="0 0 0" xyz="-0.0 -0.1 -0.05"/>
     <geometry>
-      <mesh filename="package://test_description/meshes/left_wheel_1.stl" scale="0.001 0.001 0.001"/>
+      <mesh filename="$(find test_description)/meshes/left_wheel_1.stl" scale="0.001 0.001 0.001"/>
     </geometry>
     <material name="silver"/>
@@ -81,5 +81,5 @@
     <origin rpy="0 0 0" xyz="-0.0 -0.1 -0.05"/>
     <geometry>
-      <mesh filename="package://test_description/meshes/left_wheel_1.stl" scale="0.001 0.001 0.001"/>
+      <mesh filename="$(find test_description)/meshes/left_wheel_1.stl" scale="0.001 0.001 0.001"/>
     </geometry>
   </collision>

Commit message: gazebo plugins added

File: test_description/urdf/fusionbot.urdf.xacro (robot description, xacro)
@@ -85,4 +85,56 @@
   </collision>
 </link>
+<link name="lidar_3d">
+  <pose>0 0 0 0 0 0</pose>
+</link>
+<link name="imu_link">
+  <pose>0 0 0 0 0 0</pose>
+</link>
+<link name="camera_link">
+  <pose>0 0 0 0 0 0</pose>
+</link>
+<link name="depth_camera_link">
+  <pose>0 0 0 0 0 0</pose>
+</link>
+<link name="depth_camera_optical_link">
+  <pose>0 0 0 0 0 0</pose>
+</link>
+<link name="gps_link">
+  <pose>0 0 0 0 0 0</pose>
+  <!-- <inertial>
+    <mass value="0.01"/>
+    <inertia ixx="0.01" ixy="0" ixz="0" iyy="0.01" iyz="0" izz="0.01"/>
+  </inertial> -->
+</link>
+<joint name="imu_joint" type="fixed">
+  <origin rpy="0 0 0" xyz="0.0 0.0 0.05" />
+  <parent link="base_link" />
+  <child link="imu_link" />
+  <axis xyz="0.0 0.0 0.0" />
+</joint>
+<joint name="camera_joint" type="fixed">
+  <origin rpy="0 0 0" xyz="0.1 0.0 0.05" />
+  <parent link="base_link" />
+  <child link="camera_link" />
+  <axis xyz="0.0 0.0 0.0" />
+</joint>
+<joint name="depth_camera_joint" type="fixed">
+  <origin rpy="0 0 0" xyz="0.1 0.0 0.05" />
+  <parent link="base_link" />
+  <child link="depth_camera_link" />
+  <axis xyz="0.0 0.0 0.0" />
+</joint>
+<joint name="depth_camera_optical_joint" type="fixed">
+  <origin rpy="-1.57079632679 0 -1.57079632679" xyz="0 0 0" />
+  <parent link="depth_camera_link" />
+  <child link="depth_camera_optical_link" />
+  <axis xyz="0.0 0.0 0.0" />
+</joint>
+<joint name="gps_joint" type="fixed">
+  <origin rpy="0 0 0" xyz="0.0 0.0 0.05" />
+  <parent link="base_link" />
+  <child link="gps_link" />
+  <axis xyz="0.0 0.0 0.0" />
+</joint>
 <joint name='base_link_joint' type='fixed'>
   <origin rpy="0 0 0" xyz="0 0 0" />
@@ -94,4 +146,9 @@
   <parent link="base_link"/>
   <child link="lidar_1"/>
+</joint>
+<joint name="lidar_3d_joint" type="fixed">
+  <origin rpy="0 0 0" xyz="0.05 0.0 0.11"/>
+  <parent link="lidar_1"/>
+  <child link="lidar_3d"/>
 </joint>
 <joint name="right_wheel_joint" type="continuous">
