Commit message: reordered ok

File: fusionbot_gazebo/urdf/fusionbot.urdf (robot description, URDF)
Before this commit: robot fusionbot, 11 links, 10 joints
Links:
- link base_link: geometry collision mesh filename=/home/roadbalance/ros2_ws/install/fusionbot_description/sha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 scale=0.001 0.001 0.001; visual mesh filename=/home/roadbalance/ros2_ws/install/fusionbot_description/sha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 scale=0.001 0.001 0.001
