Commit message: xacro spawn done!

File: fusionbot_description/urdf/fusionbot.urdf.xacro (robot description, xacro)
@@ -13,5 +13,5 @@
       <origin rpy="0 0 0" xyz="0 0 0" />
       <geometry>
-        <mesh filename="model://fusionbot/meshes/fusionbot/base_link.stl" scale="0.001 0.001 0.001" />
+        <mesh filename="$(find fusionbot_description)/meshes/base_link.stl" scale="0.001 0.001 0.001" />
       </geometry>
       <material name="silver" />
@@ -20,5 +20,5 @@
       <origin rpy="0 0 0" xyz="0 0 0" />
       <geometry>
-        <mesh filename="model://fusionbot/meshes/fusionbot/base_link.stl" scale="0.001 0.001 0.001" />
+        <mesh filename="$(find fusionbot_description)/meshes/base_link.stl" scale="0.001 0.001 0.001" />
       </geometry>
     </collision>
@@ -33,5 +33,5 @@
       <origin rpy="0 0 0" xyz="-0.0 0.1 -0.05" />
       <geometry>
-        <mesh filename="model://fusionbot/meshes/fusionbot/right_wheel_1.stl" scale="0.001 0.001 0.001" />
+        <mesh filename="$(find fusionbot_description)/meshes/right_wheel_1.stl" scale="0.001 0.001 0.001" />
       </geometry>
       <material name="silver" />
@@ -40,5 +40,5 @@
       <origin rpy="0 0 0" xyz="-0.0 0.1 -0.05" />
       <geometry>
-        <mesh filename="model://fusionbot/meshes/fusionbot/right_wheel_1.stl" scale="0.001 0.001 0.001" />
+        <mesh filename="$(find fusionbot_description)/meshes/right_wheel_1.stl" scale="0.001 0.001 0.001" />
       </geometry>
     </collision>
@@ -53,5 +53,5 @@
       <origin rpy="0 0 0" xyz="-0.0 -0.1 -0.05" />
       <geometry>
-        <mesh filename="model://fusionbot/meshes/fusionbot/left_wheel_1.stl" scale="0.001 0.001 0.001" />
+        <mesh filename="$(find fusionbot_description)/meshes/left_wheel_1.stl" scale="0.001 0.001 0.001" />
       </geometry>
       <material name="silver" />
@@ -60,5 +60,5 @@
       <origin rpy="0 0 0" xyz="-0.0 -0.1 -0.05" />
       <geometry>
-        <mesh filename="model://fusionbot/meshes/fusionbot/left_wheel_1.stl" scale="0.001 0.001 0.001" />
+        <mesh filename="$(find fusionbot_description)/meshes/left_wheel_1.stl" scale="0.001 0.001 0.001" />
       </geometry>
     </collision>
@@ -73,5 +73,5 @@
       <origin rpy="0 0 0" xyz="-0.05 -0.0 -0.11" />
       <geometry>
-        <mesh filename="model://fusionbot/meshes/fusionbot/lidar_1.stl" scale="0.001 0.001 0.001" />
+        <mesh filename="$(find fusionbot_description)/meshes/lidar_1.stl" scale="0.001 0.001 0.001" />
       </geometry>
       <material name="silver" />
@@ -80,5 +80,5 @@
       <origin rpy="0 0 0" xyz="-0.05 -0.0 -0.11" />
       <geometry>
-        <mesh filename="model://fusionbot/meshes/fusionbot/lidar_1.stl" scale="0.001 0.001 0.001" />
+        <mesh filename="$(find fusionbot_description)/meshes/lidar_1.stl" scale="0.001 0.001 0.001" />
       </geometry>
     </collision>

Commit message: urdf err resolved

File: fusionbot_description/urdf/fusionbot.urdf.xacro (robot description, xacro)
@@ -1,6 +1,6 @@
 <?xml version="1.0"?>
 <robot name="fusionbot" xmlns:xacro="http://www.ros.org/wiki/xacro">
-  <xacro:include filename="$(find fusionbot_description)/urdf/materials.xacro" />
-  <xacro:include filename="$(find fusionbot_description)/urdf/fusionbot.gazebo" />
+  <xacro:include filename="$(find fusionbot_gazebo)/urdf/materials.xacro" />
+  <xacro:include filename="$(find fusionbot_gazebo)/urdf/fusionbot.gazebo" />
   <link name='base_footprint' />
   <link name="base_link">

File: fusionbot_gazebo/urdf/fusionbot.urdf (robot description, URDF)
Before this commit: robot fusionbot, 11 links, 10 joints
Links:
- link base_link: geometry collision mesh filename=/home/kimsooyoung/add_ros2_ws/install/fusionbot_gazebo/shar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 scale=0.001 0.001 0.001; visual mesh filename=/home/kimsooyoung/add_ros2_ws/install/fusionbot_gazebo/shar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 scale=0.001 0.001 0.001
- link left_wheel_1: geometry collision mesh filename=/home/kimsooyoung/add_ros2_ws/install/fusionbot_gazebo/shar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 scale=0.001 0.001 0.001; visual mesh filename=/home/kimsooyoung/add_ros2_ws/install/fusionbot_gazebo/shar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 scale=0.001 0.001 0.001
- link lidar_1: geometry collision mesh filename=/home/kimsooyoung/add_ros2_ws/install/fusionbot_gazebo/shar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 scale=0.001 0.001 0.001; visual mesh filename=/home/kimsooyoung/add_ros2_ws/install/fusionbot_gazebo/shar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 scale=0.001 0.001 0.001
- link right_wheel_1: geometry collision mesh filename=/home/kimsooyoung/add_ros2_ws/install/fusionbot_gazebo/shar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 scale=0.001 0.001 0.001; visual mesh filename=/home/kimsooyoung/add_ros2_ws/install/fusionbot_gazebo/shar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 scale=0.001 0.001 0.001

File: fusionbot_gazebo/urdf/fusionbot.urdf.xacro (robot description, xacro)
@@ -1,6 +1,6 @@
 <?xml version="1.0"?>
 <robot name="fusionbot" xmlns:xacro="http://www.ros.org/wiki/xacro">
-  <xacro:include filename="$(find fusionbot_description)/urdf/materials.xacro" />
-  <xacro:include filename="$(find fusionbot_description)/urdf/fusionbot.gazebo" />
+  <xacro:include filename="$(find fusionbot_gazebo)/urdf/materials.xacro" />
+  <xacro:include filename="$(find fusionbot_gazebo)/urdf/fusionbot.gazebo" />
   <link name='base_footprint' />
   <link name="base_link">
@@ -13,5 +13,5 @@
       <origin rpy="0 0 0" xyz="0 0 0" />
       <geometry>
-        <mesh filename="$(find fusionbot_description)/meshes/base_link.stl" scale="0.001 0.001 0.001" />
+        <mesh filename="$(find fusionbot_gazebo)/meshes/base_link.stl" scale="0.001 0.001 0.001" />
       </geometry>
       <material name="silver" />
@@ -20,5 +20,5 @@
       <origin rpy="0 0 0" xyz="0 0 0" />
       <geometry>
-        <mesh filename="$(find fusionbot_description)/meshes/base_link.stl" scale="0.001 0.001 0.001" />
+        <mesh filename="$(find fusionbot_gazebo)/meshes/base_link.stl" scale="0.001 0.001 0.001" />
       </geometry>
     </collision>
@@ -33,5 +33,5 @@
       <origin rpy="0 0 0" xyz="-0.0 0.1 -0.05" />
       <geometry>
-        <mesh filename="$(find fusionbot_description)/meshes/right_wheel_1.stl" scale="0.001 0.001 0.001" />
+        <mesh filename="$(find fusionbot_gazebo)/meshes/right_wheel_1.stl" scale="0.001 0.001 0.001" />
       </geometry>
       <material name="silver" />
@@ -40,5 +40,5 @@
       <origin rpy="0 0 0" xyz="-0.0 0.1 -0.05" />
       <geometry>
-        <mesh filename="$(find fusionbot_description)/meshes/right_wheel_1.stl" scale="0.001 0.001 0.001" />
+        <mesh filename="$(find fusionbot_gazebo)/meshes/right_wheel_1.stl" scale="0.001 0.001 0.001" />
       </geometry>
     </collision>
@@ -53,5 +53,5 @@
       <origin rpy="0 0 0" xyz="-0.0 -0.1 -0.05" />
       <geometry>
-        <mesh filename="$(find fusionbot_description)/meshes/left_wheel_1.stl" scale="0.001 0.001 0.001" />
+        <mesh filename="$(find fusionbot_gazebo)/meshes/left_wheel_1.stl" scale="0.001 0.001 0.001" />
       </geometry>
       <material name="silver" />
@@ -60,5 +60,5 @@
       <origin rpy="0 0 0" xyz="-0.0 -0.1 -0.05" />
       <geometry>
-        <mesh filename="$(find fusionbot_description)/meshes/left_wheel_1.stl" scale="0.001 0.001 0.001" />
+        <mesh filename="$(find fusionbot_gazebo)/meshes/left_wheel_1.stl" scale="0.001 0.001 0.001" />
       </geometry>
     </collision>
@@ -73,5 +73,5 @@
       <origin rpy="0 0 0" xyz="-0.05 -0.0 -0.11" />
       <geometry>
-        <mesh filename="$(find fusionbot_description)/meshes/lidar_1.stl" scale="0.001 0.001 0.001" />
+        <mesh filename="$(find fusionbot_gazebo)/meshes/lidar_1.stl" scale="0.001 0.001 0.001" />
       </geometry>
       <material name="silver" />
@@ -80,5 +80,5 @@
       <origin rpy="0 0 0" xyz="-0.05 -0.0 -0.11" />
       <geometry>
-        <mesh filename="$(find fusionbot_description)/meshes/lidar_1.stl" scale="0.001 0.001 0.001" />
+        <mesh filename="$(find fusionbot_gazebo)/meshes/lidar_1.stl" scale="0.001 0.001 0.001" />
       </geometry>
     </collision>
