Commit message: ros1 gz done

File: fusionbot_gazebo_ros1/urdf/fusionbot.urdf.xacro (robot description, xacro)
@@ -85,14 +85,20 @@
   </link>
   <link name="imu_link">
-    <inertial>
-      <mass value="0.01"/>
-      <inertia ixx="0.01" ixy="0" ixz="0" iyy="0.01" iyz="0" izz="0.01"/>
-    </inertial>
+    <pose>0 0 0 0 0 0</pose>
   </link>
   <link name="camera_link">
-    <inertial>
-      <mass value="0.01"/>
-      <inertia ixx="0.01" ixy="0" ixz="0" iyy="0.01" iyz="0" izz="0.01"/>
-    </inertial>
+    <pose>0 0 0 0 0 0</pose>
+  </link>
+  <link name="depth_camera_link">
+    <pose>0 0 0 0 0 0</pose>
+  </link>
+  <link name="depth_camera_optical_link">
+    <pose>0 0 0 0 0 0</pose>
+  </link>
+  <link name="gps_link">
+    <pose>0 0 0 0 0 0</pose>
+  </link>
+  <link name="lidar_3d_link">
+    <pose>0 0 0 0 0 0</pose>
   </link>
   <joint name='base_link_joint' type='fixed'>
@@ -119,8 +125,26 @@
     <axis xyz="0.0 0.0 0.0" />
   </joint>
+  <joint name="gps_joint" type="fixed">
+    <origin rpy="0 0 0" xyz="0.0 0.0 0.05" />
+    <parent link="base_link" />
+    <child link="gps_link" />
+    <axis xyz="0.0 0.0 0.0" />
+  </joint>
   <joint name="camera_joint" type="fixed">
     <origin rpy="0 0 0" xyz="0.1 0.0 0.05" />
     <parent link="base_link" />
     <child link="camera_link" />
+    <axis xyz="0.0 0.0 0.0" />
+  </joint>
+  <joint name="depth_camera_joint" type="fixed">
+    <origin rpy="0 0 0" xyz="0 0 0" />
+    <parent link="camera_link" />
+    <child link="depth_camera_link" />
+    <axis xyz="0.0 0.0 0.0" />
+  </joint>
+  <joint name="depth_camera_optical_joint" type="fixed">
+    <origin rpy="-1.57079632679 0 -1.57079632679" xyz="0 0 0" />
+    <parent link="depth_camera_link" />
+    <child link="depth_camera_optical_link" />
     <axis xyz="0.0 0.0 0.0" />
   </joint>
@@ -130,3 +154,8 @@
     <child link="lidar_1" />
   </joint>
+  <joint name="lidar_3d_joint" type="fixed">
+    <origin rpy="0 0 0" xyz="0.05 0.0 0.11" />
+    <parent link="base_link" />
+    <child link="lidar_3d_link" />
+  </joint>
 </robot>
